Commit message: reworked xacro files to avoid duplicate content and ensure compatibility with turtlebot3_manipulator

File: open_manipulator_x_description/urdf/materials.xacro (robot description, xacro)
@@ -1,4 +1,4 @@
 <?xml version="1.0"?>
-<robot>
+<robot xmlns:xacro="http://ros.org/wiki/xacro">
   <material name="black">
     <color rgba="0.0 0.0 0.0 1.0"/>

File: open_manipulator_x_description/urdf/open_manipulator_x.gazebo.xacro (robot description, xacro)
@@ -15,77 +15,60 @@
   <!-- World -->
   <gazebo reference="world"/>
-  <!-- Link1 -->
-  <RefLink ref="link1"/>
-  <!-- Link2 -->
-  <RefLink ref="link2"/>
-  <!-- Link3 -->
-  <RefLink ref="link3"/>
-  <!-- Link4 -->
-  <RefLink ref="link4"/>
-  <!-- Link5 -->
-  <RefLink ref="link5"/>
-  <!-- gripper_link -->
-  <RefLink ref="gripper_link"/>
-  <!-- gripper_link_sub -->
-  <RefLink ref="gripper_link_sub"/>
-  <!-- end effector link -->
+  <xacro:RefLink ref="link1"/>
+  <xacro:RefLink ref="link2"/>
+  <xacro:RefLink ref="link3"/>
+  <xacro:RefLink ref="link4"/>
+  <xacro:RefLink ref="link5"/>
+  <xacro:RefLink ref="gripper_link"/>
+  <xacro:RefLink ref="gripper_link_sub"/>
   <gazebo reference="end_effector_link">
     <material>Gazebo/Red</material>
   </gazebo>
-  <!-- ros_control plugin -->
+  <!-- ros2_control plugin -->
+  <!--
+      Valid types are: position, velocity or effort
+      Recommended default MIN and MAX are:
+      position: min position, max position
+      velocity: min vel, max vel
+      effort: not sure on units... demo uses -1000 to 1000
+  -->
+  <xacro:macro name="GzJointControl" params="joint_name min max type gear_ratio">
+    <joint name="${joint_name}">
+      <command_interface name="${type}">
+        <param name="min">${min}</param>
+        <param name="max">${max}</param>
+      </command_interface>
+      <state_interface name="position"/>
+      <state_interface name="velocity"/>
+      <state_interface name="effort"/>
+    </joint>
+    <!-- It's not clear if this method of transmission definition is currently supported, but it doesn't break anything
+    and it is cleaner than other definition styles... postponing this TODO until transmissions are actually needed...
+    relevant git issue- https://github.com/ros-controls/ros2_control/issues/291 -->
+    <transmission name="${joint_name}_transmission">
+      <type>transmission_interface/SimpleTransmission</type>
+      <actuator name="${joint_name}_actuator">
+        <mechanicalReduction>${gear_ratio}</mechanicalReduction>
+      </actuator>
+      <joint name="${joint_name}">
+        <offset>0.0</offset>
+      </joint>
+    </transmission>
+  </xacro:macro>
+  <ros2_control name="GazeboSystem" type="system">
+    <hardware>
+      <plugin>gazebo_ros2_control/GazeboSystem</plugin>
+    </hardware>
+    <xacro:GzJointControl joint_name="joint1" min="-2.82743338823" max="2.82743338823" type="position" gear_ratio="1"/>
+    <xacro:GzJointControl joint_name="joint2" min="-1.79070781255" max="1.57079632679" type="position" gear_ratio="1"/>
+    <xacro:GzJointControl joint_name="joint3" min="-0.94247779607" max="1.38230076758" type="position" gear_ratio="1"/>
+    <xacro:GzJointControl joint_name="joint4" min="-1.79070781255" max="2.04203522483" type="position" gear_ratio="1"/>
+    <xacro:GzJointControl joint_name="gripper" min="-1" max="1" type="effort" gear_ratio="1"/>
+    <xacro:GzJointControl joint_name="gripper_sub" min="-1" max="1" type="effort" gear_ratio="1"/>
+  </ros2_control>
   <gazebo>
-    <plugin name="gazebo_ros_control" filename="libgazebo_ros_control.so">
-      <controlPeriod>0.001</controlPeriod>
-      <robotSimType>gazebo_ros_control/DefaultRobotHWSim</robotSimType>
+    <plugin filename="libgazebo_ros2_control.so" name="gazebo_ros2_control">
+      <parameters>$(find turtlebot3_manipulation_gazebo)/config/gz_controller.yaml</parameters>
     </plugin>
   </gazebo>
-  <!-- loading plugin: mimic joints works in gazebo now -->
-  <!-- <gazebo>
-    <plugin name="gazebo_gripper_ros_control" filename="libroboticsgroup_gazebo_mimic_joint_plugin.so">
-      <joint>gripper</joint>
-      <mimicJoint>gripper_sub</mimicJoint>
-      <multiplier>1.0</multiplier>
-      <offset>0.0</offset>
-    </plugin>
-  </gazebo> -->
-  <!-- camera -->
-  <!-- Noise is sampled independently per pixel on each frame.
-        That pixel's noise value is added to each of its color
-        channels, which at that point lie in the range [0,1]. -->
-  <!-- <gazebo reference="camera_link">
-    <sensor type="camera" name="intel_realsense_r200">
-      <update_rate>30.0</update_rate>
-      <camera name="head">
-        <horizontal_fov>1.02974</horizontal_fov>
-        <image>
-          <width>1920</width>
-          <height>1080</height>
-          <format>R8G8B8</format>
-        </image>
-        <clip>
-          <near>0.02</near>
-          <far>300</far>
-        </clip>
-        <noise>
-          <type>gaussian</type>
-          <mean>0.0</mean>
-          <stddev>0.007</stddev>
-        </noise>
-      </camera>
-      <plugin name="camera_controller" filename="libgazebo_ros_camera.so">
-        <alwaysOn>true</alwaysOn>
-        <updateRate>0.0</updateRate>
-        <cameraName>camera/color</cameraName>
-        <imageTopicName>image_raw</imageTopicName>
-        <cameraInfoTopicName>camera_info</cameraInfoTopicName>
-        <frameName>camera_link</frameName>
-        <hackBaseline>0.07</hackBaseline>
-        <distortionK1>0.0</distortionK1>
-        <distortionK2>0.0</distortionK2>
-        <distortionK3>0.0</distortionK3>
-        <distortionT1>0.0</distortionT1>
-        <distortionT2>0.0</distortionT2>
-      </plugin>
-    </sensor>
-  </gazebo> -->
 </robot>

File: open_manipulator_x_description/urdf/open_manipulator_x.transmission.xacro (robot description, xacro)
@@ -1,4 +1,6 @@
 <?xml version="1.0"?>
 <robot xmlns:xacro="http://ros.org/wiki/xacro">
+<!-- TODO: it seems like the transmissions should be specified with the joint and command interface
+           (currently in ...gazebo.xacro). This probably doesn't do anything as is.  -->
   <!-- Transmission macro -->
   <xacro:macro name="SimpleTransmissionPosition" params="joint n">

File: open_manipulator_x_description/urdf/open_manipulator_x.urdf.xacro (robot description, xacro)
@@ -6,12 +6,15 @@
       <origin xyz="0 0 0" rpy="0 0 0"/>
       <geometry>
-        <mesh filename="package://open_manipulator_x_description/meshes/chain_link1.stl" scale="0.001 0.001 0.001"/>
-      </geometry>
-      <material name="grey"/>
-    </visual>
-    <collision>
-      <origin xyz="0 0 0" rpy="0 0 0"/>
-      <geometry>
-        <mesh filename="package://open_manipulator_x_description/meshes/chain_link1.stl" scale="0.001 0.001 0.001"/>
+        <mesh filename="file://$(find open_manipulator_x_description)/meshes/chain_link1.stl" scale="0.001 0.001 0.001"/>
+      </geometry>
+      <material name="grey"/>
+    </visual>
+    <collision>
+<!--      <origin xyz="0 0 0" rpy="0 0 0"/>-->
+      <origin xyz="0 0 0.017" rpy="0 0 0"/>
+      <geometry>
+<!--        <mesh filename="file://$(find open_manipulator_x_description)/meshes/chain_link1.stl" scale="0.001 0.001 0.001"/>-->
+        <box size="0.0465 0.0285 0.034"/>
+<!--        <box size="0.0285 0.0465 0.034"/>-->
       </geometry>
     </collision>
@@ -22,4 +25,171 @@
                iyy="2.1898364e-05" iyz="0.0"
                izz="1.9267361e-05" />
+    </inertial>
+  </link>
+  <!--  Link 2 -->
+  <link name="link2">
+    <visual>
+      <origin xyz="0 0 0.019" rpy="0 0 0"/>
+      <geometry>
+        <mesh filename="file://$(find open_manipulator_x_description)/meshes/chain_link2.stl" scale="0.001 0.001 0.001"/>
+      </geometry>
+      <material name="grey"/>
+    </visual>
+    <collision>
+<!--      <origin xyz="0 0 0.019" rpy="0 0 0"/>-->
+      <origin xyz="0 0 0.05025" rpy="0 0 0"/>
+      <geometry>
+<!--        <mesh filename="file://$(find open_manipulator_x_description)/meshes/chain_link2.stl" scale="0.001 0.001 0.001"/>-->
+        <box size="0.0285 0.034 0.0625"/>
+      </geometry>
+    </collision>
+     <inertial>
+      <origin xyz="-3.0184870e-04 5.4043684e-04 0.047433464e-02" />
+      <mass value="9.8406837e-02" />
+      <inertia ixx="3.4543422e-05" ixy="-1.6031095e-08" ixz="-3.8375155e-07"
+               iyy="3.2689329e-05" iyz="2.8511935e-08"
+               izz="1.8850320e-05" />
+    </inertial>
+  </link>
+  <!--  Link 3 -->
+  <link name="link3">
+    <visual>
+      <origin xyz="0 0 0" rpy="0 0 0"/>
+      <geometry>
+        <mesh filename="file://$(find open_manipulator_x_description)/meshes/chain_link3.stl" scale="0.001 0.001 0.001"/>
+      </geometry>
+      <material name="grey"/>
+    </visual>
+    <collision>
+      <origin xyz="0.0018125 0 0.066" rpy="0 0 0"/>
+<!--      <origin xyz="0 0 0" rpy="0 0 0"/>-->
+      <geometry>
+<!--        <mesh filename="file://$(find open_manipulator_x_description)/meshes/chain_link3.stl" scale="0.001 0.001 0.001"/>-->
+        <box size="0.05875 0.052 0.172"/>
+      </geometry>
+    </collision>
+    <inertial>
+      <origin xyz="1.0308393e-02 3.7743363e-04 1.0170197e-01" />
+      <mass value="1.3850917e-01" />
+      <inertia ixx="3.3055381e-04" ixy="-9.7940978e-08" ixz="-3.8505711e-05"
+               iyy="3.4290447e-04" iyz="-1.5717516e-06"
+               izz="6.0346498e-05" />
+    </inertial>
+  </link>
+  <!--  Link 4 -->
+  <link name="link4">
+    <visual>
+      <origin xyz="0 0 0" rpy="0 0 0"/>
+      <geometry>
+        <mesh filename="file://$(find open_manipulator_x_description)/meshes/chain_link4.stl" scale="0.001 0.001 0.001"/>
+      </geometry>
+      <material name="grey"/>
+    </visual>
+    <collision>
+      <origin xyz="0.06365 0.0 0.0" rpy="0 0 0"/>
+<!--      <origin xyz="0 0 0" rpy="0 0 0"/>-->
+      <geometry>
+<!--        <mesh filename="file://$(find open_manipulator_x_description)/meshes/chain_link4.stl" scale="0.001 0.001 0.001"/>-->
+        <box size="0.1673 0.0526 0.047"/>
+      </geometry>
+    </collision>
+     <inertial>
+      <origin xyz="9.0909590e-02 3.8929816e-04 2.2413279e-04" />
+      <mass value="1.3274562e-01" />
+      <inertia ixx="3.0654178e-05" ixy="-1.2764155e-06" ixz="-2.6874417e-07"
+               iyy="2.4230292e-04" iyz="1.1559550e-08"
+               izz="2.5155057e-04" />
+    </inertial>
+  </link>
+  <!--  Link 5 -->
+  <link name="link5">
+    <visual>
+      <origin xyz="0 0 0" rpy="0 0 0"/>
+      <geometry>
+        <mesh filename="file://$(find open_manipulator_x_description)/meshes/chain_link5.stl" scale="0.001 0.001 0.001"/>
+      </geometry>
+      <material name="grey"/>
+    </visual>
+    <collision>
+      <origin xyz="0.0242 0 0.008375" rpy="0 0 0"/>
+<!--      <origin xyz="0 0 0" rpy="0 0 0"/>-->
+      <geometry>
+<!--        <mesh filename="file://$(find open_manipulator_x_description)/meshes/chain_link5.stl" scale="0.001 0.001 0.001"/>   -->
+        <box size="0.0884 0.1286  0.06275"/>
+      </geometry>
+    </collision>
+     <inertial>
+      <origin xyz="4.4206755e-02 3.6839985e-07 8.9142216e-03" />
+      <mass value="1.4327573e-01" />
+      <inertia ixx="8.0870749e-05" ixy="0.0" ixz="-1.0157896e-06"
+               iyy="7.5980465e-05" iyz="0.0"
+               izz="9.3127351e-05" />
+    </inertial>
+  </link>
+  <!--  Gripper link -->
+  <link name="gripper_link">
+    <visual>
+      <origin xyz="0.0 0.0 0" rpy="0 0 0"/>
+      <geometry>
+        <mesh filename="file://$(find open_manipulator_x_description)/meshes/chain_link_grip_l.stl" scale="0.001 0.001 0.001"/>
+      </geometry>
+      <material name="grey"/>
+    </visual>
+    <collision>
+<!--      <origin xyz="0.02095 0.00725 0" rpy="0 0 0"/>-->
+      <origin xyz="0 0 0" rpy="0 0 0"/>
+      <geometry>
+        <mesh filename="file://$(find open_manipulator_x_description)/meshes/chain_link_grip_l_low_poly.stl" scale="0.001 0.001 0.001"/>
+<!--        <box size="0.0881 0.03975 0.058"/>-->
+      </geometry>
+    </collision>
+    <inertial>
+      <origin xyz="0 0 0" />
+      <mass value="1.0e-03" />
+      <inertia ixx="1.0e-03" ixy="0.0" ixz="0.0"
+               iyy="1.0e-03" iyz="0.0"
+               izz="1.0e-03" />
+    </inertial>
+  </link>
+  <!--  Gripper link sub -->
+  <link name="gripper_link_sub">
+    <visual>
+      <origin xyz="0.0 -0.0 0" rpy="0 0 0"/>
+      <geometry>
+        <mesh filename="file://$(find open_manipulator_x_description)/meshes/chain_link_grip_r.stl" scale="0.001 0.001 0.001"/>
+      </geometry>
+      <material name="grey"/>
+    </visual>
+    <collision>
+<!--      <origin xyz="0.02095 -0.00725 0" rpy="0 0 0"/>-->
+      <origin xyz="0 0 0" rpy="0 0 0"/>
+      <geometry>
+        <mesh filename="file://$(find open_manipulator_x_description)/meshes/chain_link_grip_r_low_poly.stl" scale="0.001 0.001 0.001"/>
+<!--        <box size="0.0881 0.03975 0.058"/>-->
+      </geometry>
+    </collision>
+    <inertial>
+      <origin xyz="0 0 0" />
+      <mass value="1.0e-03" />
+      <inertia ixx="1.0e-03" ixy="0.0" ixz="0.0"
+               iyy="1.0e-03" iyz="0.0"
+               izz="1.0e-03" />
+    </inertial>
+  </link>
+  <!-- end effector link -->
+  <link name="end_effector_link">
+    <visual>
+      <origin xyz="0 0 0" rpy="0 0 0"/>
+      <geometry>
+        <box size="0.01 0.01 0.01" />
+      </geometry>
+      <material name="red"/>
+     </visual>
+    <inertial>
+      <origin xyz="0 0 0" />
+      <mass value="1.0e-03" />
+      <inertia ixx="1.0e-03" ixy="0.0" ixz="0.0"
+               iyy="1.0e-03" iyz="0.0"
+               izz="1.0e-03" />
     </inertial>
   </link>
@@ -31,28 +201,6 @@
     <axis xyz="0 0 1"/>
     <limit velocity="4.8" effort="1" lower="-2.82743338823" upper="2.82743338823" />
-  </joint>
-  <!--  Link 2 -->
-  <link name="link2">
-    <visual>
-      <origin xyz="0 0 0.019" rpy="0 0 0"/>
-      <geometry>
-        <mesh filename="package://open_manipulator_x_description/meshes/chain_link2.stl" scale="0.001 0.001 0.001"/>
-      </geometry>
-      <material name="grey"/>
-    </visual>
-    <collision>
-      <origin xyz="0 0 0.019" rpy="0 0 0"/>
-      <geometry>
-        <mesh filename="package://open_manipulator_x_description/meshes/chain_link2.stl" scale="0.001 0.001 0.001"/>
-      </geometry>
-    </collision>
-     <inertial>
-      <origin xyz="-3.0184870e-04 5.4043684e-04 0.047433464e-02" />
-      <mass value="9.8406837e-02" />
-      <inertia ixx="3.4543422e-05" ixy="-1.6031095e-08" ixz="-3.8375155e-07"
-               iyy="3.2689329e-05" iyz="2.8511935e-08"
-               izz="1.8850320e-05" />
-    </inertial>
-  </link>
+    <dynamics damping="0.2" friction="0.5"/>
+  </joint>
   <!--  Joint 2 -->
   <joint name="joint2" type="revolute">
@@ -62,28 +210,6 @@
     <axis xyz="0 1 0"/>
     <limit velocity="4.8" effort="1" lower="-1.79070781255" upper="1.57079632679" />
-  </joint>
-  <!--  Link 3 -->
-  <link name="link3">
-    <visual>
-      <origin xyz="0 0 0" rpy="0 0 0"/>
-      <geometry>
-        <mesh filename="package://open_manipulator_x_description/meshes/chain_link3.stl" scale="0.001 0.001 0.001"/>
-      </geometry>
-      <material name="grey"/>
-    </visual>
-    <collision>
-      <origin xyz="0 0 0" rpy="0 0 0"/>
-      <geometry>
-        <mesh filename="package://open_manipulator_x_description/meshes/chain_link3.stl" scale="0.001 0.001 0.001"/>
-      </geometry>
-    </collision>
-    <inertial>
-      <origin xyz="1.0308393e-02 3.7743363e-04 1.0170197e-01" />
-      <mass value="1.3850917e-01" />
-      <inertia ixx="3.3055381e-04" ixy="-9.7940978e-08" ixz="-3.8505711e-05"
-               iyy="3.4290447e-04" iyz="-1.5717516e-06"
-               izz="6.0346498e-05" />
-    </inertial>
-  </link>
+    <dynamics damping="0.2" friction="0.5"/>
+  </joint>
   <!--  Joint 3 -->
   <joint name="joint3" type="revolute">
@@ -93,28 +219,6 @@
     <axis xyz="0 1 0"/>
     <limit velocity="4.8" effort="1" lower="-0.94247779607" upper="1.38230076758" />
-  </joint>
-  <!--  Link 4 -->
-  <link name="link4">
-    <visual>
-      <origin xyz="0 0 0" rpy="0 0 0"/>
-      <geometry>
-        <mesh filename="package://open_manipulator_x_description/meshes/chain_link4.stl" scale="0.001 0.001 0.001"/>
-      </geometry>
-      <material name="grey"/>
-    </visual>
-    <collision>
-      <origin xyz="0 0 0" rpy="0 0 0"/>
-      <geometry>
-        <mesh filename="package://open_manipulator_x_description/meshes/chain_link4.stl" scale="0.001 0.001 0.001"/>
-      </geometry>
-    </collision>
-     <inertial>
-      <origin xyz="9.0909590e-02 3.8929816e-04 2.2413279e-04" />
-      <mass value="1.3274562e-01" />
-      <inertia ixx="3.0654178e-05" ixy="-1.2764155e-06" ixz="-2.6874417e-07"
-               iyy="2.4230292e-04" iyz="1.1559550e-08"
-               izz="2.5155057e-04" />
-    </inertial>
-  </link>
+    <dynamics damping="0.2" friction="0.5"/>
+  </joint>
   <!--  Joint 4 -->
   <joint name="joint4" type="revolute">
@@ -124,28 +228,6 @@
     <axis xyz="0 1 0"/>
     <limit velocity="4.8" effort="1" lower="-1.79070781255" upper="2.04203522483" />
-  </joint>
-  <!--  Link 5 -->
-  <link name="link5">
-    <visual>
-      <origin xyz="0 0 0" rpy="0 0 0"/>
-      <geometry>
-        <mesh filename="package://open_manipulator_x_description/meshes/chain_link5.stl" scale="0.001 0.001 0.001"/>
-      </geometry>
-      <material name="grey"/>
-    </visual>
-    <collision>
-      <origin xyz="0 0 0" rpy="0 0 0"/>
-      <geometry>
-        <mesh filename="package://open_manipulator_x_description/meshes/chain_link5.stl" scale="0.001 0.001 0.001"/>
-      </geometry>
-    </collision>
-     <inertial>
-      <origin xyz="4.4206755e-02 3.6839985e-07 8.9142216e-03" />
-      <mass value="1.4327573e-01" />
-      <inertia ixx="8.0870749e-05" ixy="0.0" ixz="-1.0157896e-06"
-               iyy="7.5980465e-05" iyz="0.0"
-               izz="9.3127351e-05" />
-    </inertial>
-  </link>
+    <dynamics damping="0.2" friction="0.5"/>
+  </joint>
   <!--  Gripper joint -->
   <joint name="gripper" type="prismatic">
@@ -155,28 +237,6 @@
     <axis xyz="0 1 0"/>
     <limit velocity="4.8" effort="1" lower="-0.010" upper="0.019" />
-  </joint>
-  <!--  Gripper link -->
-  <link name="gripper_link">
-    <visual>
-      <origin xyz="0.0 0.0 0" rpy="0 0 0"/>
-      <geometry>
-        <mesh filename="package://open_manipulator_x_description/meshes/chain_link_grip_l.stl" scale="0.001 0.001 0.001"/>
-      </geometry>
-      <material name="grey"/>
-    </visual>
-    <collision>
-      <origin xyz="0.0 0.0 0" rpy="0 0 0"/>
-      <geometry>
-        <mesh filename="package://open_manipulator_x_description/meshes/chain_link_grip_l.stl" scale="0.001 0.001 0.001"/>
-      </geometry>
-    </collision>
-    <inertial>
-      <origin xyz="0 0 0" />
-      <mass value="1.0e-03" />
-      <inertia ixx="1.0e-03" ixy="0.0" ixz="0.0"
-               iyy="1.0e-03" iyz="0.0"
-               izz="1.0e-03" />
-    </inertial>
-  </link>
+    <dynamics damping="0.2" friction="0.5"/>
+  </joint>
   <!--  Gripper joint sub -->
   <joint name="gripper_sub" type="prismatic">
@@ -186,29 +246,6 @@
     <axis xyz="0 -1 0"/>
     <limit velocity="4.8" effort="1" lower="-0.010" upper="0.019" />
-    <mimic joint="gripper" multiplier="1"/>
-  </joint>
-  <!--  Gripper link sub -->
-  <link name="gripper_link_sub">
-    <visual>
-      <origin xyz="0.0 -0.0 0" rpy="0 0 0"/>
-      <geometry>
-        <mesh filename="package://open_manipulator_x_description/meshes/chain_link_grip_r.stl" scale="0.001 0.001 0.001"/>
-      </geometry>
-      <material name="grey"/>
-    </visual>
-    <collision>
-      <origin xyz="0.0 -0.0 0" rpy="0 0 0"/>
-      <geometry>
-        <mesh filename="package://open_manipulator_x_description/meshes/chain_link_grip_r.stl" scale="0.001 0.001 0.001"/>
-      </geometry>
-    </collision>
-    <inertial>
-      <origin xyz="0 0 0" />
-      <mass value="1.0e-03" />
-      <inertia ixx="1.0e-03" ixy="0.0" ixz="0.0"
-               iyy="1.0e-03" iyz="0.0"
-               izz="1.0e-03" />
-    </inertial>
-  </link>
+    <dynamics damping="0.2" friction="0.5"/>
+  </joint>
   <!-- end effector joint -->
   <joint name="end_effector_joint" type="fixed">
@@ -217,28 +254,3 @@
     <child link="end_effector_link"/>
   </joint>
-  <!-- end effector link -->
-  <link name="end_effector_link">
-    <visual>
-      <origin xyz="0 0 0" rpy="0 0 0"/>
-      <geometry>
-        <box size="0.01 0.01 0.01" />
-      </geometry>
-      <material name="red"/>
-     </visual>
-    <inertial>
-      <origin xyz="0 0 0" />
-      <mass value="1.0e-03" />
-      <inertia ixx="1.0e-03" ixy="0.0" ixz="0.0"
-               iyy="1.0e-03" iyz="0.0"
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