Commit message: xacro updates

File: open_manipulator_x_description/urdf/open_manipulator_x.gazebo.xacro (robot description, xacro)
@@ -5,7 +5,7 @@
     <gazebo reference="${ref}">
       <kp>1000000.0</kp>
-      <kd>100.0</kd>
-      <mu1>30.0</mu1>
-      <mu2>30.0</mu2>
+      <kd>1.0</kd>
+      <mu1>3.0</mu1>
+      <mu2>3.0</mu2>
       <maxVel>1.0</maxVel>
       <minDepth>0.001</minDepth>
@@ -22,4 +22,10 @@
   <xacro:RefLink ref="gripper_link"/>
   <xacro:RefLink ref="gripper_link_sub"/>
+  <gazebo reference="gripper">
+    <implicitSpringDamper>1</implicitSpringDamper>
+  </gazebo>
+  <gazebo reference="gripper_sub">
+    <implicitSpringDamper>1</implicitSpringDamper>
+  </gazebo>
   <gazebo reference="end_effector_link">
     <material>Gazebo/Red</material>
@@ -67,8 +73,14 @@
     <xacro:GzJointControl joint_name="gripper_sub" min="-1" max="1" type="effort" gear_ratio="1"/>
   </ros2_control>
-  <gazebo>
-    <plugin filename="libgazebo_ros2_control.so" name="gazebo_ros2_control">
-      <parameters>$(find turtlebot3_manipulation_gazebo)/config/gz_controller.yaml</parameters>
-    </plugin>
-  </gazebo>
+  <xacro:arg name="run_arm_control" default="True"/>
+  <xacro:if value="$(arg run_arm_control)">
+    <gazebo>
+      <plugin filename="libgazebo_ros2_control.so" name="gazebo_ros2_control">
+  <!--      <ros>-->
+  <!--        <namespace>TODO</namespace>-->
+  <!--      </ros>-->
+        <parameters>$(find turtlebot3_manipulation_gazebo)/config/gz_controller.yaml</parameters>
+      </plugin>
+    </gazebo>
+  </xacro:if>
 </robot>

File: open_manipulator_x_description/urdf/open_manipulator_x.urdf.xacro (robot description, xacro)
@@ -143,8 +143,24 @@
 <!--        <box size="0.0881 0.03975 0.058"/>-->
       </geometry>
+      <surface>
+          <friction>
+            <ode>
+              <mu>100</mu>
+              <mu2>100</mu2>
+            </ode>
+          </friction>
+          <contact>
+            <ode>
+              <max_vel>.1</max_vel>
+              <min_depth>0.003</min_depth>
+<!--              <kp>1e6</kp>-->
+<!--              <kd>1e1</kd>-->
+            </ode>
+          </contact>
+      </surface>
     </collision>
     <inertial>
       <origin xyz="0 0 0" />
-      <mass value="1.0e-03" />
+      <mass value="1.0e-02" />
       <inertia ixx="1.0e-03" ixy="0.0" ixz="0.0"
                iyy="1.0e-03" iyz="0.0"
@@ -168,4 +184,20 @@
 <!--        <box size="0.0881 0.03975 0.058"/>-->
       </geometry>
+      <surface>
+          <friction>
+            <ode>
+              <mu>100</mu>
+              <mu2>100</mu2>
+            </ode>
+          </friction>
+          <contact>
+            <ode>
+              <max_vel>.1</max_vel>
+              <min_depth>0.003</min_depth>
+<!--              <kp>1e6</kp>-->
+<!--              <kd>1e1</kd>-->
+            </ode>
+          </contact>
+      </surface>
     </collision>
     <inertial>

Commit message: add hardware control support to xacro

File: open_manipulator_x_description/urdf/open_manipulator_x.gazebo.xacro (robot description, xacro)
@@ -31,56 +31,3 @@
     <material>Gazebo/Red</material>
   </gazebo>
-  <!-- ros2_control plugin -->
-  <!--
-      Valid types are: position, velocity or effort
-      Recommended default MIN and MAX are:
-      position: min position, max position
-      velocity: min vel, max vel
-      effort: not sure on units... demo uses -1000 to 1000
-  -->
-  <xacro:macro name="GzJointControl" params="joint_name min max type gear_ratio">
-    <joint name="${joint_name}">
-      <command_interface name="${type}">
-        <param name="min">${min}</param>
-        <param name="max">${max}</param>
-      </command_interface>
-      <state_interface name="position"/>
-      <state_interface name="velocity"/>
-      <state_interface name="effort"/>
-    </joint>
-    <!-- It's not clear if this method of transmission definition is currently supported, but it doesn't break anything
-    and it is cleaner than other definition styles... postponing this TODO until transmissions are actually needed...
-    relevant git issue- https://github.com/ros-controls/ros2_control/issues/291 -->
-    <transmission name="${joint_name}_transmission">
-      <type>transmission_interface/SimpleTransmission</type>
-      <actuator name="${joint_name}_actuator">
-        <mechanicalReduction>${gear_ratio}</mechanicalReduction>
-      </actuator>
-      <joint name="${joint_name}">
-        <offset>0.0</offset>
-      </joint>
-    </transmission>
-  </xacro:macro>
-  <ros2_control name="GazeboSystem" type="system">
-    <hardware>
-      <plugin>gazebo_ros2_control/GazeboSystem</plugin>
-    </hardware>
-    <xacro:GzJointControl joint_name="joint1" min="-2.82743338823" max="2.82743338823" type="position" gear_ratio="1"/>
-    <xacro:GzJointControl joint_name="joint2" min="-1.79070781255" max="1.57079632679" type="position" gear_ratio="1"/>
-    <xacro:GzJointControl joint_name="joint3" min="-0.94247779607" max="1.38230076758" type="position" gear_ratio="1"/>
-    <xacro:GzJointControl joint_name="joint4" min="-1.79070781255" max="2.04203522483" type="position" gear_ratio="1"/>
-    <xacro:GzJointControl joint_name="gripper" min="-1" max="1" type="effort" gear_ratio="1"/>
-    <xacro:GzJointControl joint_name="gripper_sub" min="-1" max="1" type="effort" gear_ratio="1"/>
-  </ros2_control>
-  <xacro:arg name="run_arm_control" default="True"/>
-  <xacro:if value="$(arg run_arm_control)">
-    <gazebo>
-      <plugin filename="libgazebo_ros2_control.so" name="gazebo_ros2_control">
-  <!--      <ros>-->
-  <!--        <namespace>TODO</namespace>-->
-  <!--      </ros>-->
-        <parameters>$(find turtlebot3_manipulation_gazebo)/config/gz_controller.yaml</parameters>
-      </plugin>
-    </gazebo>
-  </xacro:if>
 </robot>
