Commit message: xacro cleanup

File: open_manipulator_x_description/urdf/open_manipulator_x.controller.xacro (robot description, xacro)
@@ -1,76 +1,71 @@
 <?xml version="1.0"?>
 <robot xmlns:xacro="http://ros.org/wiki/xacro">
-  <xacro:arg name="run_arm_control" default="True"/>
   <xacro:if value="$(arg run_arm_control)">
-  <!-- ros2_control plugin -->
-  <!--
-      Valid types are: position, velocity or effort
-      Recommended default MIN and MAX are:
-      position: min position, max position
-      velocity: min vel, max vel
-      effort: not sure on units... demo uses -1000 to 1000
-  -->
-  <xacro:macro name="ros2_control_macro" params="joint_name min max type gear_ratio secondary_interface:=''">
-    <joint name="${joint_name}">
-      <command_interface name="${type}">
-        <param name="min">${min}</param>
-        <param name="max">${max}</param>
-      </command_interface>
-      <xacro:if value="${secondary_interface != ''}">
-        <command_interface name="${secondary_interface}"/>
+    <!-- ros2_control plugin -->
+    <!--
+        Valid types are: position, velocity or effort
+        Recommended default MIN and MAX are:
+        position: min position, max position
+        velocity: min vel, max vel
+        effort: not sure on units... demo uses -1000 to 1000
+    -->
+    <xacro:macro name="ros2_control_macro" params="joint_name min max type gear_ratio secondary_interface:=''">
+      <joint name="${joint_name}">
+        <command_interface name="${type}">
+          <param name="min">${min}</param>
+          <param name="max">${max}</param>
+        </command_interface>
+        <xacro:if value="${secondary_interface != ''}">
+          <command_interface name="${secondary_interface}"/>
+        </xacro:if>
+        <state_interface name="position"/>
+        <state_interface name="velocity"/>
+        <state_interface name="effort"/>
+      </joint>
+      <!-- It's not clear if this method of transmission definition is currently supported, but it doesn't break anything
+      and it is cleaner than other definition styles... postponing this TODO until transmissions are actually needed...
+      relevant git issue- https://github.com/ros-controls/ros2_control/issues/291 -->
+      <transmission name="${joint_name}_transmission">
+        <type>transmission_interface/SimpleTransmission</type>
+        <actuator name="${joint_name}_actuator">
+          <mechanicalReduction>${gear_ratio}</mechanicalReduction>
+        </actuator>
+        <joint name="${joint_name}">
+          <offset>0.0</offset>
+        </joint>
+      </transmission>
+    </xacro:macro>
+    <ros2_control name="open_manipulator_x_ros2_control" type="system">
+      <xacro:if value="$(arg gazebo)">
+        <hardware>
+          <plugin>gazebo_ros2_control/GazeboSystem</plugin>
+        </hardware>
+        <xacro:ros2_control_macro joint_name="joint1" min="-2.82743338823" max="2.82743338823" type="position" gear_ratio="1"/>
+        <xacro:ros2_control_macro joint_name="joint2" min="-1.79070781255" max="1.57079632679" type="position" gear_ratio="1"/>
+        <xacro:ros2_control_macro joint_name="joint3" min="-0.94247779607" max="1.38230076758" type="position" gear_ratio="1"/>
+        <xacro:ros2_control_macro joint_name="joint4" min="-1.79070781255" max="2.04203522483" type="position" gear_ratio="1"/>
+        <xacro:ros2_control_macro joint_name="gripper" min="-1" max="1" type="effort" gear_ratio="1"/>
+        <xacro:ros2_control_macro joint_name="gripper_sub" min="-1" max="1" type="effort" gear_ratio="1"/>
       </xacro:if>
-      <state_interface name="position"/>
-      <state_interface name="velocity"/>
-      <state_interface name="effort"/>
-    </joint>
-    <!-- It's not clear if this method of transmission definition is currently supported, but it doesn't break anything
-    and it is cleaner than other definition styles... postponing this TODO until transmissions are actually needed...
-    relevant git issue- https://github.com/ros-controls/ros2_control/issues/291 -->
-    <transmission name="${joint_name}_transmission">
-      <type>transmission_interface/SimpleTransmission</type>
-      <actuator name="${joint_name}_actuator">
-        <mechanicalReduction>${gear_ratio}</mechanicalReduction>
-      </actuator>
-      <joint name="${joint_name}">
-        <offset>0.0</offset>
-      </joint>
-    </transmission>
-  </xacro:macro>
-  <ros2_control name="open_manipulator_x_ros2_control" type="system">
-    <!-- ======================================================================== -->
-    <!-- ======================================================================== -->
-    <xacro:if value="$(arg gazebo)">
-      <hardware>
-        <plugin>gazebo_ros2_control/GazeboSystem</plugin>
-      </hardware>
-      <xacro:ros2_control_macro joint_name="joint1" min="-2.82743338823" max="2.82743338823" type="position" gear_ratio="1"/>
-      <xacro:ros2_control_macro joint_name="joint2" min="-1.79070781255" max="1.57079632679" type="position" gear_ratio="1"/>
-      <xacro:ros2_control_macro joint_name="joint3" min="-0.94247779607" max="1.38230076758" type="position" gear_ratio="1"/>
-      <xacro:ros2_control_macro joint_name="joint4" min="-1.79070781255" max="2.04203522483" type="position" gear_ratio="1"/>
-      <xacro:ros2_control_macro joint_name="gripper" min="-1" max="1" type="effort" gear_ratio="1"/>
-      <xacro:ros2_control_macro joint_name="gripper_sub" min="-1" max="1" type="effort" gear_ratio="1"/>
-    </xacro:if>
-    <xacro:if value="${not $(arg gazebo)}">
-      <hardware>
-        <plugin>dynamixel_hardware/DynamixelHardware</plugin>
-        <param name="usb_port">/dev/ttyUSB1</param>
-        <param name="baud_rate">1000000</param>
-        <param name="joint_ids">11,12,13,14,15</param>
-      </hardware>
-      <xacro:ros2_control_macro joint_name="joint1" min="-2.82743338823" max="2.82743338823" type="position" gear_ratio="1"/>
-      <xacro:ros2_control_macro joint_name="joint2" min="-1.79070781255" max="1.57079632679" type="position" gear_ratio="1"/>
-      <xacro:ros2_control_macro joint_name="joint3" min="-0.94247779607" max="1.38230076758" type="position" gear_ratio="1"/>
-      <xacro:ros2_control_macro joint_name="joint4" min="-1.79070781255" max="2.04203522483" type="position" gear_ratio="1"/>
-      <xacro:ros2_control_macro joint_name="gripper" min="-0.01" max="0.01" type="position" gear_ratio="1"/>
-    </xacro:if>
-    <!-- ======================================================================== -->
-    <!-- ======================================================================== -->
+      <xacro:if value="${not $(arg gazebo)}">
+        <hardware>
+          <plugin>dynamixel_hardware/DynamixelHardware</plugin>
+          <param name="usb_port">/dev/ttyUSB1</param>
+          <param name="baud_rate">1000000</param>
+          <param name="joint_ids">11,12,13,14,15</param>
+        </hardware>
+        <xacro:ros2_control_macro joint_name="joint1" min="-2.82743338823" max="2.82743338823" type="position" gear_ratio="1"/>
+        <xacro:ros2_control_macro joint_name="joint2" min="-1.79070781255" max="1.57079632679" type="position" gear_ratio="1"/>
+        <xacro:ros2_control_macro joint_name="joint3" min="-0.94247779607" max="1.38230076758" type="position" gear_ratio="1"/>
+        <xacro:ros2_control_macro joint_name="joint4" min="-1.79070781255" max="2.04203522483" type="position" gear_ratio="1"/>
+        <xacro:ros2_control_macro joint_name="gripper" min="-0.01" max="0.01" type="position" gear_ratio="1"/>
+      </xacro:if>
     </ros2_control>
     <xacro:if value="$(arg gazebo)">
       <gazebo>
         <plugin filename="libgazebo_ros2_control.so" name="gazebo_ros2_control">
-  <!--      <ros>-->
-  <!--        <namespace>TODO</namespace>-->
-  <!--      </ros>-->
+          <!--      <ros>-->
+          <!--        <namespace>TODO</namespace>-->
+          <!--      </ros>-->
           <parameters>$(find turtlebot3_manipulation_gazebo)/config/gz_controller.yaml</parameters>
         </plugin>

File: open_manipulator_x_description/urdf/open_manipulator_x_robot.urdf.xacro (robot description, xacro)
@@ -2,8 +2,14 @@
 <!-- OpenManipulator Chain -->
 <robot name="open_manipulator_x" xmlns:xacro="http://ros.org/wiki/xacro">
+  <xacro:arg name="run_arm_control" default="True"/>
+  <xacro:arg name="gazebo" default="True"/>
   <!-- Import Rviz colors -->
   <xacro:include filename="$(find open_manipulator_x_description)/urdf/materials.xacro" />
   <!-- Import all Gazebo-customization elements, including Gazebo colors -->
-  <xacro:include filename="$(find open_manipulator_x_description)/urdf/open_manipulator_x.gazebo.xacro" />
+  <xacro:if value="$(arg gazebo)">
+    <xacro:include filename="$(find open_manipulator_x_description)/urdf/open_manipulator_x.gazebo.xacro" />
+  </xacro:if>
+  <!-- Import ROS2 Control elements -->
+  <xacro:include filename="$(find open_manipulator_x_description)/urdf/open_manipulator_x.controller.xacro" />
   <!-- Import Transmission -->
   <xacro:include filename="$(find open_manipulator_x_description)/urdf/open_manipulator_x.transmission.xacro" />
